File: hardware/Menorah.sch (KiCad schematic (older format))
At the start: 26 parts, among them SW1 SW_Push, U1 ATtiny85-20PU

Commit message: assigned footprints, started layout
Parts:
- removed BT1, BT2, BT3, BT4, BT5, BT6: Battery_Cell, Battery:BatteryHolder_Keystone_3000_1x12mm, symbol Device:Battery_Cell
- added BT1: Battery, Connector_PinHeader_1.27mm:PinHeader_1x02_P1.27mm_Vertical_SMD_Pin1Left, symbol Device:Battery
Connections:
- wire segments 93 -> 73
- no-connect marks 0 -> 2
Changed lines of the file:
@@
 	6700 1950 6700 1350
-$Comp
-L Device:Battery_Cell BT1
-U 1 1 5DE7F2D8
-P 1650 1700
-F 0 "BT1" H 1768 1796 50  0000 L CNN
-F 1 "Battery_Cell" H 1768 1705 50  0000 L CNN
-F 2 "Battery:BatteryHolder_Keystone_3000_1x12mm" V 1650 1760 50  0001 C CNN
-F 3 "~" V 1650 1760 50  0001 C CNN
-	1    1650 1700
-	1    0    0    -1
-$EndComp
-$Comp
-L Device:Battery_Cell BT4
-U 1 1 5DE7FBBF
-P 1650 2300
-F 0 "BT4" H 1768 2396 50  0000 L CNN
-F 1 "Battery_Cell" H 1768 2305 50  0000 L CNN
-F 2 "Battery:BatteryHolder_Keystone_3000_1x12mm" V 1650 2360 50  0001 C CNN
-F 3 "~" V 1650 2360 50  0001 C CNN
-	1    1650 2300
-	1    0    0    -1
-$EndComp
-Wire Wire Line
-	2300 1500 2300 1400
-Wire Wire Line
-	2300 1400 1650 1400
-Wire Wire Line
-	1650 1400 1650 1500
-Wire Wire Line
-	2300 1800 2300 1900
-Wire Wire Line
-	2300 1900 1650 1900
-Wire Wire Line
-	1650 1900 1650 1800
-$Comp
-L Device:Battery_Cell BT2
-U 1 1 5DE841C4
-P 2300 1700
-F 0 "BT2" H 2418 1796 50  0000 L CNN
-F 1 "Battery_Cell" H 2418 1705 50  0000 L CNN
-F 2 "Battery:BatteryHolder_Keystone_3000_1x12mm" V 2300 1760 50  0001 C CNN
-F 3 "~" V 2300 1760 50  0001 C CNN
-	1    2300 1700
-	1    0    0    -1
-$EndComp
-$Comp
-L Device:Battery_Cell BT5
-U 1 1 5DE841CA
-P 2300 2300
-F 0 "BT5" H 2418 2396 50  0000 L CNN
-F 1 "Battery_Cell" H 2418 2305 50  0000 L CNN
-F 2 "Battery:BatteryHolder_Keystone_3000_1x12mm" V 2300 2360 50  0001 C CNN
-F 3 "~" V 2300 2360 50  0001 C CNN
-	1    2300 2300
-	1    0    0    -1
-$EndComp
-$Comp
-L Device:Battery_Cell BT3
-U 1 1 5DE865A6
-P 2950 1700
-F 0 "BT3" H 3068 1796 50  0000 L CNN
-F 1 "Battery_Cell" H 3068 1705 50  0000 L CNN
-F 2 "Battery:BatteryHolder_Keystone_3000_1x12mm" V 2950 1760 50  0001 C CNN
-F 3 "~" V 2950 1760 50  0001 C CNN
-	1    2950 1700
-	1    0    0    -1
-$EndComp
-$Comp
-L Device:Battery_Cell BT6
-U 1 1 5DE865AC
-P 2950 2300
-F 0 "BT6" H 3068 2396 50  0000 L CNN
-F 1 "Battery_Cell" H 3068 2305 50  0000 L CNN
-F 2 "Battery:BatteryHolder_Keystone_3000_1x12mm" V 2950 2360 50  0001 C CNN
-F 3 "~" V 2950 2360 50  0001 C CNN
-	1    2950 2300
-	1    0    0    -1
-$EndComp
 $Comp
 L power:GND #PWR01
 U 1 1 5DE8FC9F
-P 1650 2500
-F 0 "#PWR01" H 1650 2250 50  0001 C CNN
-F 1 "GND" H 1655 2327 50  0000 C CNN
-F 2 "" H 1650 2500 50  0001 C CNN
-F 3 "" H 1650 2500 50  0001 C CNN
-	1    1650 2500
-	1    0    0    -1
-$EndComp
-Wire Wire Line
-	4100 1300 4250 1300
+P 2950 2300
+F 0 "#PWR01" H 2950 2050 50  0001 C CNN
+F 1 "GND" H 2955 2127 50  0000 C CNN
+F 2 "" H 2950 2300 50  0001 C CNN
+F 3 "" H 2950 2300 50  0001 C CNN
+	1    2950 2300
+	1    0    0    -1
+$EndComp
 Wire Wire Line
 	4650 1300 4950 1300
@@
 Wire Wire Line
 	5650 1300 5500 1300
-Wire Wire Line
-	2300 1400 2950 1400
-Wire Wire Line
-	2950 1400 2950 1500
-Connection ~ 2300 1400
-Wire Wire Line
-	2300 1900 2950 1900
-Wire Wire Line
-	2950 1900 2950 1800
-Connection ~ 2300 1900
-Wire Wire Line
-	1650 2100 1650 2000
-Wire Wire Line
-	1650 2000 2300 2000
-Wire Wire Line
-	2300 2000 2300 2100
-Wire Wire Line
-	2300 2000 2950 2000
-Wire Wire Line
-	2950 2000 2950 2100
-Connection ~ 2300 2000
-Wire Wire Line
-	1650 2400 1650 2500
-Wire Wire Line
-	1650 2500 2300 2500
-Wire Wire Line
-	2300 2500 2300 2400
-Wire Wire Line
-	2300 2500 2950 2500
-Wire Wire Line
-	2950 2500 2950 2400
-Connection ~ 2300 2500
-Wire Wire Line
-	1650 1900 1650 2000
-Connection ~ 1650 1900
-Connection ~ 1650 2000
-Connection ~ 1650 2500
-Wire Wire Line
-	2950 1400 3700 1400
-Connection ~ 2950 1400
 Connection ~ 8800 2350
 Wire Wire Line
@@
 Wire Wire Line
 	4950 2750 4950 3150
+$Comp
+L Device:Battery BT1
+U 1 1 5FB7AD5A
+P 2950 1850
+F 0 "BT1" H 3058 1896 50  0000 L CNN
+F 1 "Battery" H 3058 1805 50  0000 L CNN
+F 2 "Connector_PinHeader_1.27mm:PinHeader_1x02_P1.27mm_Vertical_SMD_Pin1Left" V 2950 1910 50  0001 C CNN
+F 3 "~" V 2950 1910 50  0001 C CNN
+	1    2950 1850
+	1    0    0    -1
+$EndComp
+Wire Wire Line
+	2950 1650 2950 1300
+Wire Wire Line
+	2950 1300 4250 1300
+Wire Wire Line
+	2950 2050 2950 2300
+NoConn ~ 5550 2350
+NoConn ~ 6000 3850
 $EndSCHEMATC

Commit message: lotsa stuff
Parts:
- removed D10, D11, D12: LED, LED_SMD:LED_1206_3216Metric, symbol Device:LED
- added D10, D11, D12: 1N4004, Diode_SMD:D_SOD-123F, symbol pspice:DIODE
- added J1: Conn_02x03_Odd_Even, Connector_PinHeader_2.54mm:PinHeader_2x03_P2.54mm_Vertical_SMD, symbol Connector_Generic:Conn_02x03_Odd_Even
- renumbered D7 to D6, D6 to D7
Connections:
- net GND: now also J1.6 (Pin_6)
- net at D1.2 (A), D2.1 (K), D7.2 (A)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: now also D11.1 (K), D12.2 (A)
- net at D1.1 (K), D2.2 (A), D3.2 (A)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: now also D10.2 (A)
- net at D5.1 (K), D6.2 (A), D9.1 (K)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: now also D10.1 (K), D11.2 (A), D12.1 (K)
- net RST: now reaches U1.1 (~RESET~/PB5)
- net RST: now also J1.5 (Pin_5)
- net MOSI: now reaches R5.1, SW1.1, U1.5 (AREF/PB0)
- net MOSI: now also J1.4 (Pin_4)
- net MISO: now reaches R1.2, U1.6 (PB1)
- net MISO: now also J1.1 (Pin_1)
- net SCK: now reaches R2.2, U1.7 (PB2)
- net SCK: now also J1.3 (Pin_3)
- net VCC: now reaches D13.2 (A), R5.2, U1.8 (VCC)
- net VCC: now also J1.2 (Pin_2)
- no-connect marks 2 -> 0
Changed lines of the file:
@@
 EESchema Schematic File Version 4
+LIBS:Menorah-cache
 EELAYER 30 0
 EELAYER END
@@
 	6700 2250 6700 2850
 Wire Wire Line
-	5550 1950 6700 1950
+	5550 1950 5600 1950
 Wire Wire Line
 	6700 1950 6700 1350
@@
 	8800 2350 9150 2350
 Wire Wire Line
-	9150 2850 8800 2850
-Wire Wire Line
-	9500 2850 9150 2850
-Wire Wire Line
-	9150 1350 9500 1350
-Wire Wire Line
-	9150 1350 8800 1350
-Wire Wire Line
 	7400 1350 7750 1350
 Wire Wire Line
@@
 Wire Wire Line
 	6800 2050 6800 1850
-Wire Wire Line
-	5550 2050 6800 2050
 Connection ~ 8100 2850
 $Comp
@@
 $EndComp
 Connection ~ 8800 1350
-Connection ~ 9150 1350
-Connection ~ 9150 2850
 Wire Wire Line
 	9150 1850 9150 1750
 Wire Wire Line
 	9500 1750 9500 1850
-Wire Wire Line
-	9150 1350 9150 1450
-Wire Wire Line
-	9500 1350 9500 1450
-$Comp
-L Device:LED D10
-U 1 1 5DE594C4
-P 9150 1600
-F 0 "D10" V 9189 1483 50  0000 R CNN
-F 1 "LED" V 9098 1483 50  0000 R CNN
-F 2 "LED_SMD:LED_1206_3216Metric" H 9150 1600 50  0001 C CNN
-F 3 "~" H 9150 1600 50  0001 C CNN
-	1    9150 1600
-	0    -1   -1   0
-$EndComp
-$Comp
-L Device:LED D12
-U 1 1 5DE594BE
-P 9500 1600
-F 0 "D12" V 9447 1678 50  0000 L CNN
-F 1 "LED" V 9538 1678 50  0000 L CNN
-F 2 "LED_SMD:LED_1206_3216Metric" H 9500 1600 50  0001 C CNN
-F 3 "~" H 9500 1600 50  0001 C CNN
-	1    9500 1600
-	0    1    1    0
-$EndComp
 Connection ~ 8100 1850
 Wire Wire Line
@@
 	8800 2850 8800 2750
 Wire Wire Line
-	9150 2750 9150 2850
-Wire Wire Line
 	8800 2350 8800 2450
-Wire Wire Line
-	9150 2350 9150 2450
 $Comp
 L Device:LED D9
@@
 	0    -1   -1   0
 $EndComp
-$Comp
-L Device:LED D11
-U 1 1 5DE56237
-P 9150 2600
-F 0 "D11" V 9097 2678 50  0000 L CNN
-F 1 "LED" V 9188 2678 50  0000 L CNN
-F 2 "LED_SMD:LED_1206_3216Metric" H 9150 2600 50  0001 C CNN
-F 3 "~" H 9150 2600 50  0001 C CNN
-	1    9150 2600
-	0    1    1    0
-$EndComp
 Connection ~ 8450 2350
 Connection ~ 8450 1850
@@
 	8800 1350 8800 1450
 $Comp
-L Device:LED D6
+L Device:LED D7
 U 1 1 5DE4E7B5
 P 8450 1600
-F 0 "D6" V 8489 1483 50  0000 R CNN
+F 0 "D7" V 8489 1483 50  0000 R CNN
 F 1 "LED" V 8398 1483 50  0000 R CNN
 F 2 "LED_SMD:LED_1206_3216Metric" H 8450 1600 50  0001 C CNN
@@
 $EndComp
 $Comp
-L Device:LED D7
+L Device:LED D6
 U 1 1 5DE45951
 P 8450 2600
-F 0 "D7" V 8397 2678 50  0000 L CNN
+F 0 "D6" V 8397 2678 50  0000 L CNN
 F 1 "LED" V 8488 2678 50  0000 L CNN
 F 2 "LED_SMD:LED_1206_3216Metric" H 8450 2600 50  0001 C CNN
@@
 $EndComp
 Wire Wire Line
-	4950 1550 4950 1300
+	4950 1550 4950 1450
 $Comp
 L Device:R R5
@@
 Wire Wire Line
 	2950 2050 2950 2300
-NoConn ~ 5550 2350
-NoConn ~ 6000 3850
+$Comp
+L pspice:DIODE D11
+U 1 1 5FB893C9
+P 9150 1550
+F 0 "D11" H 9150 1815 50  0000 C CNN
+F 1 "1N4004" H 9150 1724 50  0000 C CNN
+F 2 "Diode_SMD:D_SOD-123F" H 9150 1550 50  0001 C CNN
+F 3 "~" H 9150 1550 50  0001 C CNN
+	1    9150 1550
+	0    1    1    0
+$EndComp
+$Comp
+L pspice:DIODE D12
+U 1 1 5FB8AD89
+P 9500 1550
+F 0 "D12" H 9500 1815 50  0000 C CNN
+F 1 "1N4004" H 9500 1724 50  0000 C CNN
+F 2 "Diode_SMD:D_SOD-123F" H 9500 1550 50  0001 C CNN
+F 3 "~" H 9500 1550 50  0001 C CNN
+	1    9500 1550
+	0    1    -1   0
+$EndComp
+$Comp
+L pspice:DIODE D10
+U 1 1 5FB8C7CB
+P 9150 2600
+F 0 "D10" H 9150 2865 50  0000 C CNN
+F 1 "1N4004" H 9150 2774 50  0000 C CNN
+F 2 "Diode_SMD:D_SOD-123F" H 9150 2600 50  0001 C CNN
+F 3 "~" H 9150 2600 50  0001 C CNN
+	1    9150 2600
+	0    1    -1   0
+$EndComp
+Wire Wire Line
+	8800 1350 9150 1350
+Connection ~ 9150 1350
+Wire Wire Line
+	9150 1350 9500 1350
+Wire Wire Line
+	8800 2850 9150 2850
+Wire Wire Line
+	9150 2800 9150 2850
+Connection ~ 9150 2850
+Wire Wire Line
+	9150 2850 9500 2850
+Wire Wire Line
+	9150 2400 9150 2350
+$Comp
+L Connector_Generic:Conn_02x03_Odd_Even J1
+U 1 1 5FBC1514
+P 3450 2950
+F 0 "J1" H 3500 3267 50  0000 C CNN
+F 1 "Conn_02x03_Odd_Even" H 3500 3176 50  0000 C CNN
+F 2 "Connector_PinHeader_2.54mm:PinHeader_2x03_P2.54mm_Vertical_SMD" H 3450 2950 50  0001 C CNN
+F 3 "~" H 3450 2950 50  0001 C CNN
+	1    3450 2950
+	1    0    0    -1
+$EndComp
+Text GLabel 3150 2850 0    50   Input ~ 0
+MISO
+Wire Wire Line
+	3150 2850 3250 2850
+Text GLabel 3150 2950 0    50   Input ~ 0
+SCK
+Wire Wire Line
+	3150 2950 3250 2950
+Text GLabel 3150 3050 0    50   Input ~ 0
+RST
+Wire Wire Line
+	3150 3050 3250 3050
+Text GLabel 3850 2850 2    50   Input ~ 0
+VCC
+Text GLabel 3850 2950 2    50   Input ~ 0
+MOSI
+Wire Wire Line
+	3850 2950 3750 2950
+Wire Wire Line
+	3850 2850 3750 2850
+Text GLabel 5650 2350 2    50   Input ~ 0
+RST
+Wire Wire Line
+	5650 2350 5550 2350
+$Comp
+L power:GND #PWR03
+U 1 1 5FBD5DFC
+P 3950 3100
+F 0 "#PWR03" H 3950 2850 50  0001 C CNN
+F 1 "GND" H 3955 2927 50  0000 C CNN
+F 2 "" H 3950 3100 50  0001 C CNN
+F 3 "" H 3950 3100 50  0001 C CNN
+	1    3950 3100
+	1    0    0    -1
+$EndComp
+Wire Wire Line
+	3950 3100 3950 3050
+Wire Wire Line
+	3750 3050 3950 3050
+Text GLabel 6150 2100 2    50   Input ~ 0
+SCK
+Text GLabel 5650 2000 2    50   Input ~ 0
+MISO
+Wire Wire Line
+	5650 2000 5600 2000
+Wire Wire Line
+	5600 2000 5600 1950
+Connection ~ 5600 1950
+Wire Wire Line
+	5600 1950 6700 1950
+Text GLabel 5750 1850 2    50   Input ~ 0
+MOSI
+Wire Wire Line
+	5750 1850 5650 1850
+Connection ~ 5650 1850
+Wire Wire Line
+	5550 2050 6100 2050
+Wire Wire Line
+	6150 2100 6100 2100
+Wire Wire Line
+	6100 2100 6100 2050
+Connection ~ 6100 2050
+Wire Wire Line
+	6100 2050 6800 2050
+Text GLabel 5050 1450 2    50   Input ~ 0
+VCC
+Wire Wire Line
+	5050 1450 4950 1450
+Connection ~ 4950 1450
+Wire Wire Line
+	4950 1450 4950 1300
 $EndSCHEMATC

Commit message: Added BOM
Parts:
- R1, R2, R3, R4: value 68 -> 51
Other:
- moved on the sheet: D12
Changed lines of the file:
@@
 	8800 1850 8450 1850
-Wire Wire Line
-	9500 1850 9150 1850
 Wire Wire Line
 	8450 1350 8800 1350
@@
 P 6950 2850
 F 0 "R4" V 6743 2850 50  0000 C CNN
-F 1 "68" V 6834 2850 50  0000 C CNN
+F 1 "51" V 6834 2850 50  0000 C CNN
 F 2 "Resistor_SMD:R_0805_2012Metric" V 6880 2850 50  0001 C CNN
 F 3 "~" H 6950 2850 50  0001 C CNN
@@
 P 6950 2350
 F 0 "R3" V 6743 2350 50  0000 C CNN
-F 1 "68" V 6834 2350 50  0000 C CNN
+F 1 "51" V 6834 2350 50  0000 C CNN
 F 2 "Resistor_SMD:R_0805_2012Metric" V 6880 2350 50  0001 C CNN
 F 3 "~" H 6950 2350 50  0001 C CNN
@@
 P 6950 1850
 F 0 "R2" V 6743 1850 50  0000 C CNN
-F 1 "68" V 6834 1850 50  0000 C CNN
+F 1 "51" V 6834 1850 50  0000 C CNN
 F 2 "Resistor_SMD:R_0805_2012Metric" V 6880 1850 50  0001 C CNN
 F 3 "~" H 6950 1850 50  0001 C CNN
@@
 P 6950 1350
 F 0 "R1" V 6743 1350 50  0000 C CNN
-F 1 "68" V 6834 1350 50  0000 C CNN
+F 1 "51" V 6834 1350 50  0000 C CNN
 F 2 "Resistor_SMD:R_0805_2012Metric" V 6880 1350 50  0001 C CNN
 F 3 "~" H 6950 1350 50  0001 C CNN
@@
 Wire Wire Line
 	9150 1850 9150 1750
-Wire Wire Line
-	9500 1750 9500 1850
 Connection ~ 8100 1850
 Wire Wire Line
@@
 Wire Wire Line
 	8450 1850 8450 2350
-Connection ~ 9500 1850
-Wire Wire Line
-	9500 1850 9500 2850
 $Comp
 L power:GND #PWR0101
@@
 L pspice:DIODE D12
 U 1 1 5FB8AD89
-P 9500 1550
-F 0 "D12" H 9500 1815 50  0000 C CNN
-F 1 "1N4004" H 9500 1724 50  0000 C CNN
-F 2 "Diode_SMD:D_SOD-123F" H 9500 1550 50  0001 C CNN
-F 3 "~" H 9500 1550 50  0001 C CNN
-	1    9500 1550
+P 9550 1550
+F 0 "D12" H 9550 1815 50  0000 C CNN
+F 1 "1N4004" H 9550 1724 50  0000 C CNN
+F 2 "Diode_SMD:D_SOD-123F" H 9550 1550 50  0001 C CNN
+F 3 "~" H 9550 1550 50  0001 C CNN
+	1    9550 1550
 	0    1    -1   0
 $EndComp
@@
 Connection ~ 9150 1350
 Wire Wire Line
-	9150 1350 9500 1350
-Wire Wire Line
 	8800 2850 9150 2850
 Wire Wire Line
 	9150 2800 9150 2850
 Connection ~ 9150 2850
-Wire Wire Line
-	9150 2850 9500 2850
 Wire Wire Line
 	9150 2400 9150 2350
@@
 Wire Wire Line
 	4950 1450 4950 1300
+Wire Wire Line
+	9150 1350 9550 1350
+Wire Wire Line
+	9550 1750 9550 1850
+Wire Wire Line
+	9150 1850 9550 1850
+Connection ~ 9550 1850
+Wire Wire Line
+	9550 1850 9550 2850
+Wire Wire Line
+	9150 2850 9550 2850
 $EndSCHEMATC
